Commit message: Enable camera in the main urdf, changed the depth camera for new gazebo

File: models/my_robot_description/depth_camera.xacro (robot description, xacro)
@@ -9,12 +9,8 @@
   <link name="depth_camera_back_link">
     <visual>
-      <geometry>
-        <box size="0.0016 0.085 0.024"/>
-      </geometry>
+      <geometry><box size="0.0016 0.085 0.024"/></geometry>
     </visual>
     <collision>
-      <geometry>
-        <box size="0.0016 0.085 0.024"/>
-      </geometry>
+      <geometry><box size="0.0016 0.085 0.024"/></geometry>
     </collision>
     <xacro:inertial_box mass="0.05" x="0.0016" y="0.085" z="0.024">
@@ -22,23 +18,17 @@
     </xacro:inertial_box>
   </link>
-  <gazebo reference="depth_camera_back_link">
-    <material>Gazebo/White</material>
-  </gazebo>
-  <!-- Left camera cylinder -->
+  <gazebo reference="depth_camera_back_link"><material>Gazebo/White</material></gazebo>
+  <!-- ================= LEFT CAMERA ================= -->
   <joint name="left_camera_joint" type="fixed">
     <parent link="depth_camera_back_link"/>
     <child link="left_camera_link"/>
-    <origin xyz="0.0058 -0.036 0" rpy="0 0 0"/> <!-- Rotate to length along x (forward), baseline along y -->
+    <origin xyz="0.0058 -0.036 0" rpy="0 0 0"/>
   </joint>
   <link name="left_camera_link">
     <visual>
-      <geometry>
-        <box size = "0.01 0.0155 0.0155"/> <!-- Length along x (forward) -->
-      </geometry>
+      <geometry><box size = "0.01 0.0155 0.0155"/></geometry>
     </visual>
     <collision>
-      <geometry>
-        <box size = "0.01 0.0155 0.0155"/>
-      </geometry>
+      <geometry><box size = "0.01 0.0155 0.0155"/></geometry>
     </collision>
     <xacro:inertial_box mass="0.02" x="0.01" y="0.0155" z="0.0155">
@@ -48,10 +38,12 @@
   <gazebo reference="left_camera_link">
     <material>Gazebo/Black</material>
+    <!-- IGNITION FORTRESS SENSOR TAG -->
     <sensor type="camera" name="left_camera">
       <always_on>true</always_on>
       <visualize>true</visualize>
       <update_rate>30</update_rate>
+      <topic>depth_cam/left/image_raw</topic>
       <camera>
-        <horizontal_fov>1.044815127601244</horizontal_fov>
+        <horizontal_fov>1.0448151276</horizontal_fov>
         <image>
           <width>640</width>
@@ -63,47 +55,26 @@
           <far>50.0</far>
         </clip>
-        <!--<noise>
-          <type>gaussian</type>
-          <mean>0.0</mean>
-          <stddev>0.01</stddev>
-        </noise>-->
       </camera>
-      <plugin name="left_camera_controller" filename="libgazebo_ros_camera.so">
-        <ros>
-          <namespace>/follower_robot</namespace>
-        </ros>
-        <camera_name>depth_cam/left</camera_name>
-        <frame_name>left_camera_link_optical</frame_name>
-        <!--<focal_length>1424.1969168622516</focal_length>
-        <cx>812.6941986083984</cx>
-        <cy>615.3056335449219</cy>
-        <cx_prime>812.6941986083984</cx_prime>
-        <hack_baseline>0.0</hack_baseline>-->
-      </plugin>
     </sensor>
   </gazebo>
-  <!-- Left optical frame (view from front flat base) -->
+  <!-- Left optical frame -->
   <joint name="left_camera_optical_joint" type="fixed">
     <parent link="left_camera_link"/>
     <child link="left_camera_link_optical"/>
-    <origin xyz="0.01 0 0" rpy="${-pi/2} 0 ${-pi/2}"/> <!-- Shift to front flat (+0.01 x), rotate for ROS optical convention -->
+    <origin xyz="0.01 0 0" rpy="${-pi/2} 0 ${-pi/2}"/>
   </joint>
   <link name="left_camera_link_optical"/>
-  <!-- Right camera cylinder -->
+  <!-- ================= RIGHT CAMERA ================= -->
   <joint name="right_camera_joint" type="fixed">
     <parent link="depth_camera_back_link"/>
     <child link="right_camera_link"/>
-    <origin xyz="0.0058 0.036 0" rpy="0 0 0"/> <!-- Rotate to length along x (forward), baseline along y -->
+    <origin xyz="0.0058 0.036 0" rpy="0 0 0"/>
   </joint>
   <link name="right_camera_link">
     <visual>
-      <geometry>
-        <box size = "0.01 0.0155 0.0155"/> <!-- Length along x (forward) -->
-      </geometry>
+      <geometry><box size = "0.01 0.0155 0.0155"/></geometry>
     </visual>
     <collision>
-      <geometry>
-        <box size = "0.01 0.0155 0.0155"/>
-      </geometry>
+      <geometry><box size = "0.01 0.0155 0.0155"/></geometry>
     </collision>
     <xacro:inertial_box mass="0.02" x="0.01" y="0.0155" z="0.0155">
@@ -113,10 +84,12 @@
   <gazebo reference="right_camera_link">
     <material>Gazebo/Black</material>
+    <!-- IGNITION FORTRESS SENSOR TAG -->
     <sensor type="camera" name="right_camera">
       <always_on>true</always_on>
       <visualize>true</visualize>
       <update_rate>30</update_rate>
+      <topic>depth_cam/right/image_raw</topic>
       <camera>
-        <horizontal_fov>1.044815127601244</horizontal_fov>
+        <horizontal_fov>1.0448151276</horizontal_fov>
         <image>
           <width>640</width>
@@ -128,35 +101,13 @@
           <far>50.0</far>
         </clip>
-        <!--<noise>
-          <type>gaussian</type>
-          <mean>0.0</mean>
-          <stddev>0.01</stddev>
-        </noise>-->
       </camera>
-      <plugin name="right_camera_controller" filename="libgazebo_ros_camera.so">
-        <ros>
-          <namespace>/follower_robot</namespace>
-        </ros>
-        <camera_name>depth_cam/right</camera_name>  <!-- Sets prefix for topics: /depth_cam/right/image_raw and /depth_cam/right/camera_info -->
-        <frame_name>right_camera_link_optical</frame_name>
-        <!--<focal_length>1424.1969168622516</focal_length>
-        <cx>812.6941986083984</cx>
-        <cy>615.3056335449219</cy>
-        <cx_prime>812.6941986083984</cx_prime>-->
-        <hack_baseline>-0.071727</hack_baseline>
-      </plugin>
     </sensor>
   </gazebo>
-  <!-- Right optical frame (view from front flat base) -->
+  <!-- Right optical frame -->
   <joint name="right_camera_optical_joint" type="fixed">
     <parent link="right_camera_link"/>
     <child link="right_camera_link_optical"/>
-    <origin xyz="0.01 0 0" rpy="${-pi/2} 0 ${-pi/2}"/> <!-- Shift to front flat (+0.01 x), rotate for ROS optical convention -->
+    <origin xyz="0.01 0 0" rpy="${-pi/2} 0 ${-pi/2}"/>
   </joint>
   <link name="right_camera_link_optical"/>
-  <plugin name="clock_sync" filename="libgazebo_ros_clock.so">
-    <ros>
-      <namespace>/</namespace>
-    </ros>
-  </plugin>
 </robot>

File: models/my_robot_description/my_robot.urdf.xacro (robot description, xacro)
@@ -4,4 +4,4 @@
     <xacro:include filename="gazebo_control.xacro"/>
     <!--<xacro:include filename="stereo_camera.xacro"/>-->
-    <!--xacro:include filename="depth_camera.xacro"/-->
+    <xacro:include filename="depth_camera.xacro"/>
 </robot>

Commit message: modified files

File: models/my_robot_description/depth_camera.xacro (robot description, xacro)
@@ -32,5 +32,5 @@
     <parent link="depth_camera_back_link"/>
     <child link="left_camera_link"/>
-    <origin xyz="0.0058 -0.036 0" rpy="0 0 0"/>
+    <origin xyz="0.0058 -0.03 0" rpy="0 0 0"/>
   </joint>
   <link name="left_camera_link">
@@ -55,5 +55,5 @@
       <topic>depth_cam/left</topic>
       <camera>
-        <horizontal_fov>1.0448151276</horizontal_fov>
+        <horizontal_fov>1.27409</horizontal_fov>
         <image>
           <width>640</width>
@@ -63,6 +63,17 @@
         <clip>
           <near>0.02</near>
-          <far>50.0</far>
+          <far>8.0</far>
         </clip>
+        <lens>
+          <intrinsics>
+            <!-- fx = fy = width / (2 * tan(horizontal_fov/2)), computed for horizontal_fov=1.27409, width=640 -->
+            <fx>432.43</fx>
+            <fy>432.43</fy>
+            <!-- cx = (width-1)/2, cy = (height-1)/2 -->
+            <cx>319.5</cx>
+            <cy>239.5</cy>
+            <s>0</s>
+          </intrinsics>
+        </lens>
       </camera>
     </sensor>
@@ -79,5 +90,5 @@
     <parent link="depth_camera_back_link"/>
     <child link="right_camera_link"/>
-    <origin xyz="0.0058 0.036 0" rpy="0 0 0"/>
+    <origin xyz="0.0058 0.03 0" rpy="0 0 0"/>
   </joint>
   <link name="right_camera_link">
@@ -102,5 +113,5 @@
       <topic>depth_cam/right</topic>
       <camera>
-        <horizontal_fov>1.0448151276</horizontal_fov>
+        <horizontal_fov>1.27409</horizontal_fov>
         <image>
           <width>640</width>
@@ -110,6 +121,17 @@
         <clip>
           <near>0.02</near>
-          <far>50.0</far>
+          <far>8.0</far>
         </clip>
+        <lens>
+          <intrinsics>
+            <!-- fx = fy = width / (2 * tan(horizontal_fov/2)), computed for horizontal_fov=1.27409, width=640 -->
+            <fx>432.43</fx>
+            <fy>432.43</fy>
+            <!-- cx = (width-1)/2, cy = (height-1)/2 -->
+            <cx>319.5</cx>
+            <cy>239.5</cy>
+            <s>0</s>
+          </intrinsics>
+        </lens>
       </camera>
     </sensor>
